File: Servo_Controller/ServoController.kicad_sch (KiCad schematic)
At the start: 42 parts, among them J1 USB_B_Micro, K1 SWD, K2 Signal/Power, M1 Motor, U1 STM32F103C8T6, U2 TPD2E001DZDR, U3 AMS1117-3.3, U4 IRS4427S, U5 AO4616, U6 AO4616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

Commit message: Added enclosure, removed unnecessary resistor
Parts:
- removed R1: 4.7k, ServoController:R_0402, symbol Device:R
Connections:
- net USB_DET: no longer names the net of U1.46 (PB9/TIM4_CH4(RTOP)/I2C1_SDA/CANTX)
- no-connect marks 29 -> 30
Changed lines of the file:
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@@
   (no_connect (at 91.44 212.09))
   (no_connect (at 165.1 97.79))
+  (no_connect (at 58.42 110.49))
   (wire (pts (xy 185.42 57.15) (xy 185.42 59.69))
     (stroke (width 0) (type default) (color 0 0 0 0))
@@
     (stroke (width 0) (type default) (color 0 0 0 0))
   )
-  (wire (pts (xy 91.44 195.58) (xy 78.74 195.58))
-    (stroke (width 0) (type default) (color 0 0 0 0))
-  )
   (wire (pts (xy 201.93 110.49) (xy 201.93 113.03))
     (stroke (width 0) (type default) (color 0 0 0 0))
@@
     (stroke (width 0) (type default) (color 0 0 0 0))
   )
-  (wire (pts (xy 58.42 110.49) (xy 38.1 110.49))
-    (stroke (width 0) (type default) (color 0 0 0 0))
-  )
   (wire (pts (xy 260.35 196.85) (xy 260.35 194.31))
     (stroke (width 0) (type default) (color 0 0 0 0))
@@
   )
   (wire (pts (xy 165.1 74.93) (xy 207.01 74.93))
-    (stroke (width 0) (type default) (color 0 0 0 0))
-  )
-  (wire (pts (xy 99.06 195.58) (xy 101.6 195.58))
     (stroke (width 0) (type default) (color 0 0 0 0))
   )
@@
     (effects (font (size 1.27 1.27)) (justify right bottom))
   )
-  (label "USB_DET" (at 39.37 110.49 0)
-    (effects (font (size 1.27 1.27)) (justify left bottom))
-  )
   (label "USB_DP" (at 147.32 207.01 180)
     (effects (font (size 1.27 1.27)) (justify right bottom))
-  )
-  (label "USB_DET" (at 80.01 195.58 0)
-    (effects (font (size 1.27 1.27)) (justify left bottom))
   )
   (label "MOTOR_A" (at 39.37 44.45 0)
@@
     )
     (pin "1")
-  )
-  (symbol (lib_id "Device:R") (at 95.25 195.58 90) (mirror x) (unit 1)
-    (in_bom yes) (on_board yes)
-    (property "Reference" "R1" (id 0) (at 95.25 193.04 90))
-    (property "Value" "4.7k" (id 1) (at 95.25 195.58 90))
-    (property "Footprint" "ServoController:R_0402" (id 2) (at 95.25 193.802 90)
-      (effects (font (size 1.27 1.27)) hide)
-    )
-    (property "Datasheet" "~" (id 3) (at 95.25 195.58 0)
-      (effects (font (size 1.27 1.27)) hide)
-    )
-    (pin "1")
-    (pin "2")
   )
   (symbol (lib_id "power:GND") (at 274.32 123.19 90) (unit 1)
@@
       (reference "M1") (unit 1) (value "Motor") (footprint "ServoController:Motor")
     )
-    (path "/00000000-0000-0000-0000-00006159a6c7"
-      (reference "R1") (unit 1) (value "4.7k") (footprint "ServoController:R_0402")
-    )
     (path "/00000000-0000-0000-0000-0000611bf6de"

Commit message: Changed VCC to SWO signal on SWD header. Manufacturing data and PCB previews updated
Connections:
- net GND: now also K1.1; no longer K1.5
- net MCU_SWCLK: now also K1.5; no longer K1.4
- net VCC: no longer K1.1
- net MCU_SWO: now reaches U1.39 (PB3/JTDO/TIM2_CH2/TRACESWO/SPI1_SCK)
- net MCU_SWO: now also K1.4
- no-connect marks 30 -> 29
Changed lines of the file:
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@@
   (no_connect (at 81.28 217.17))
   (no_connect (at 58.42 64.77))
-  (no_connect (at 58.42 95.25))
   (no_connect (at 58.42 125.73))
   (no_connect (at 58.42 87.63))
@@
     (stroke (width 0) (type default) (color 0 0 0 0))
   )
+  (wire (pts (xy 38.1 95.25) (xy 58.42 95.25))
+    (stroke (width 0) (type default) (color 0 0 0 0))
+  )
   (wire (pts (xy 377.19 115.57) (xy 374.65 115.57))
     (stroke (width 0) (type default) (color 0 0 0 0))
@@
     (effects (font (size 1.27 1.27)) (justify left bottom))
   )
-  (label "MCU_SWCLK" (at 102.87 144.78 0)
+  (label "MCU_SWO" (at 102.87 144.78 0)
+    (effects (font (size 1.27 1.27)) (justify left bottom))
+  )
+  (label "MCU_SWCLK" (at 102.87 147.32 0)
     (effects (font (size 1.27 1.27)) (justify left bottom))
   )
@@
   (label "VIN" (at 300.99 54.61 180)
     (effects (font (size 1.27 1.27)) (justify right bottom))
+  )
+  (label "MCU_SWO" (at 39.37 95.25 0)
+    (effects (font (size 1.27 1.27)) (justify left bottom))
   )
   (label "POTENTIOMETER" (at 386.08 137.16 180)
@@
     (pin "1")
   )
-  (symbol (lib_id "power:GND") (at 101.6 147.32 270) (mirror x) (unit 1)
-    (in_bom yes) (on_board yes)
-    (property "Reference" "#PWR03" (id 0) (at 95.25 147.32 0)
-      (effects (font (size 1.27 1.27)) hide)
-    )
-    (property "Value" "GND" (id 1) (at 99.06 147.32 90)
+  (symbol (lib_id "power:GND") (at 101.6 137.16 270) (mirror x) (unit 1)
+    (in_bom yes) (on_board yes)
+    (property "Reference" "#PWR03" (id 0) (at 95.25 137.16 0)
+      (effects (font (size 1.27 1.27)) hide)
+    )
+    (property "Value" "GND" (id 1) (at 99.06 137.16 90)
       (effects (font (size 1.27 1.27)) (justify right))
     )
-    (property "Footprint" "" (id 2) (at 101.6 147.32 0)
-      (effects (font (size 1.27 1.27)) hide)
-    )
-    (property "Datasheet" "" (id 3) (at 101.6 147.32 0)
+    (property "Footprint" "" (id 2) (at 101.6 137.16 0)
+      (effects (font (size 1.27 1.27)) hide)
+    )
+    (property "Datasheet" "" (id 3) (at 101.6 137.16 0)
       (effects (font (size 1.27 1.27)) hide)
     )
@@
     )
     (property "Datasheet" "" (id 3) (at 382.27 180.34 0)
-      (effects (font (size 1.27 1.27)) hide)
-    )
-    (pin "1")
-  )
-  (symbol (lib_id "power:VCC") (at 101.6 137.16 90) (mirror x) (unit 1)
-    (in_bom yes) (on_board yes)
-    (property "Reference" "#PWR02" (id 0) (at 105.41 137.16 0)
-      (effects (font (size 1.27 1.27)) hide)
-    )
-    (property "Value" "VCC" (id 1) (at 99.06 137.16 90)
-      (effects (font (size 1.27 1.27)) (justify left))
-    )
-    (property "Footprint" "" (id 2) (at 101.6 137.16 0)
-      (effects (font (size 1.27 1.27)) hide)
-    )
-    (property "Datasheet" "" (id 3) (at 101.6 137.16 0)
       (effects (font (size 1.27 1.27)) hide)
     )
@@
       (reference "#PWR01") (unit 1) (value "GND") (footprint "")
     )
-    (path "/00000000-0000-0000-0000-0000613bc236"
-      (reference "#PWR02") (unit 1) (value "VCC") (footprint "")
-    )
     (path "/00000000-0000-0000-0000-0000611cd553"
